Commit message: Update g1_12dof.urdf

File: resources/robots/g1/g1_12dof.urdf (robot description, URDF)
Before this commit: robot g1_12dof, 31 links, 30 joints
Joints:
- joint left_elbow_joint: origin xyz=0.015783 0 -0.080518 rpy=0 0 0 -> xyz=0.015783 0 -0.080518 rpy=0 1.3 0
- joint left_shoulder_roll_joint: origin xyz=0 0.038 -0.013831 rpy=-0.27925 0 0 -> xyz=0 0.038 -0.013831 rpy=-0.2 0 0
- joint right_elbow_joint: origin xyz=0.015783 0 -0.080518 rpy=0 0 0 -> xyz=0.015783 0 -0.080518 rpy=0 1.3 0
- joint right_shoulder_roll_joint: origin xyz=0 -0.038 -0.013831 rpy=0.27925 0 0 -> xyz=0 -0.038 -0.013831 rpy=0.2 0 0

Commit message: 2025-4-3

File: resources/robots/g1/g1_12dof.urdf (robot description, URDF)
Before this commit: robot g1_12dof, 31 links, 30 joints
Joints:
- joint left_shoulder_roll_joint: origin xyz=0 0.038 -0.013831 rpy=-0.2 0 0 -> xyz=0 0.038 -0.013831 rpy=-0 0 0
- joint right_shoulder_roll_joint: origin xyz=0 -0.038 -0.013831 rpy=0.2 0 0 -> xyz=0 -0.038 -0.013831 rpy=0 0 0

Commit message: Update g1_12dof.urdf

File: resources/robots/g1/g1_12dof.urdf (robot description, URDF)
Before this commit: robot g1_12dof, 31 links, 30 joints
Joints:
- joint left_elbow_joint: origin xyz=0.015783 0 -0.080518 rpy=0 1.3 0 -> xyz=0.015783 0 -0.080518 rpy=0 0.8 0
- joint left_shoulder_roll_joint: origin xyz=0 0.038 -0.013831 rpy=-0 0 0 -> xyz=0 0.038 -0.013831 rpy=-0.27925 0 0
- joint right_elbow_joint: origin xyz=0.015783 0 -0.080518 rpy=0 1.3 0 -> xyz=0.015783 0 -0.080518 rpy=0 0.8 0
- joint right_shoulder_roll_joint: origin xyz=0 -0.038 -0.013831 rpy=0 0 0 -> xyz=0 -0.038 -0.013831 rpy=0.27925 0 0
